Commit message: pre-flight commit

File: description/robot_core.xacro (robot description, xacro)
@@ -18,5 +18,12 @@
     </material>
     <!-- BASE LINK -->
-    <link name="base_link">
+    <link name="base_link"></link>
+    <!-- BASE_FOOTPRINT LINK -->
+    <joint name="base_footprint_joint" type="fixed">
+        <parent link="base_link"/>
+        <child link="base_footprint"/>
+        <origin xyz="0 0 0" rpy="0 0 0"/>
+    </joint>
+    <link name="base_footprint">
     </link>
     <!-- CHASSIS LINK -->

Commit message: camera cringe

File: description/robot_core.xacro (robot description, xacro)
@@ -25,6 +25,5 @@
         <origin xyz="0 0 0" rpy="0 0 0"/>
     </joint>
-    <link name="base_footprint">
-    </link>
+    <link name="base_footprint"></link>
     <!-- CHASSIS LINK -->
     <joint name="chassis_joint" type="fixed">
