Commit message: spawn both?

File: description/camera_uav.xacro (robot description, xacro)
@@ -37,5 +37,5 @@
             <origin xyz="0 0 0.005"/>
             <geometry>
-                <box size="0.3 0.3 0.01"/>
+                <box size="0.5 0.5 0.01"/>
             </geometry>
         </collision>

File: description/uav.urdf.xacro (robot description, xacro)
@@ -1,5 +1,5 @@
 <?xml version="1.0"?>
 <robot xmlns:xacro="http://www.ros.org/wiki/xacro"  name="robot">
-    <xacro:include filename="camera.xacro" />
+    <xacro:include filename="camera_uav.xacro" />
     <!-- <xacro:include filename="gazebo_control.xacro" /> -->
     <!-- <xacro:include filename="depth_camera.xacro" /> -->

Commit message: both spawn

File: description/camera_uav.xacro (robot description, xacro)
@@ -37,5 +37,5 @@
             <origin xyz="0 0 0.005"/>
             <geometry>
-                <box size="0.5 0.5 0.01"/>
+                <box size="0.3 0.3 0.01"/>
             </geometry>
         </collision>

File: description/uav.urdf.xacro (robot description, xacro)
@@ -1,4 +1,4 @@
 <?xml version="1.0"?>
-<robot xmlns:xacro="http://www.ros.org/wiki/xacro"  name="robot">
+<robot xmlns:xacro="http://www.ros.org/wiki/xacro"  name="uav">
     <xacro:include filename="camera_uav.xacro" />
     <!-- <xacro:include filename="gazebo_control.xacro" /> -->

Commit message: Dual spawn - waypoint?

File: description/camera_uav.xacro (robot description, xacro)
@@ -37,5 +37,5 @@
             <origin xyz="0 0 0.005"/>
             <geometry>
-                <box size="0.5 0.5 0.01"/>
+                <box size="0.1 0.1 0.01"/>
             </geometry>
         </collision>
@@ -84,4 +84,5 @@
             </camera>
             <plugin name="uav_camera_controller" filename="libgazebo_ros_camera.so">
+                <!-- <ros><namespace>/uav</namespace></ros> -->
                 <frame_name>camera_link_optical_uav</frame_name>
             </plugin>

File: description/lidar.xacro (robot description, xacro)
@@ -41,7 +41,8 @@
                 </range>
             </ray>
-            <plugin name="laser_controller" filename="libgazebo_ros_ray_sensor.so">
+            <plugin name="laser_controller____" filename="libgazebo_ros_ray_sensor.so">
                 <ros>
                     <argument>~/out:=scan</argument>
+                    <!-- <namespace>/ugv</namespace> -->
                 </ros>
                 <output_type>sensor_msgs/LaserScan</output_type>

File: description/robot.urdf.xacro (robot description, xacro)
@@ -10,5 +10,5 @@
     <xacro:include filename="robot_core.xacro" />
     <xacro:include filename="lidar.xacro" />
-    <xacro:include filename="camera.xacro" />
+    <!-- <xacro:include filename="camera.xacro" /> -->
     <!-- <xacro:include filename="gazebo_control.xacro" /> -->
     <!-- <xacro:include filename="depth_camera.xacro" /> -->

File: description/uav.urdf.xacro (robot description, xacro)
@@ -1,5 +1,6 @@
 <?xml version="1.0"?>
 <robot xmlns:xacro="http://www.ros.org/wiki/xacro"  name="uav">
-    <xacro:include filename="camera_uav.xacro" />
+    <!-- <xacro:include filename="camera_uav.xacro" /> -->
+    <xacro:include filename="uav.xacro" />
     <!-- <xacro:include filename="depth_camera_uav.xacro" /> -->
 </robot>
